File: KiCad/bios_kbc_rtc.kicad_sch (KiCad schematic)
At the start: 44 parts, among them J10 BANK1, J11 PS/2 Dual Port, J7 BANK0, J8 BANK0, J9 BANK1, U4 DS12885, U5 8242KBD, U6 SST39SF010A, U7 74HC05, Y2 32768Hz

Commit message: Fix the ROM /OE issue; Update DRAM banks
Connect Flash ROM /OE to ISA /MEMR
Update DRAM banks numbers (swap Bank 0 and Bank 1)
Update chipset DRAM signal names
Renumber DRAM termination resistors according to the signal names
Renumber SIMM and ISA slots, so that they are numbered top to bottom
Parts:
- J1: renamed from J10; value BANK1 -> BANK0
- J2: renamed from J9; value BANK1 -> BANK0
- J3: renamed from J8; value BANK0 -> BANK1
- J4: renamed from J7; value BANK0 -> BANK1
- renumbered R17 to R16, R16 to R17, R21 to R18, R20 to R19, R19 to R20, R18 to R21
Connections:
- net ~{MCAS0}: now also R18.1; no longer R21.1
- net ~{MCAS1}: now also R19.1; no longer R20.1
- net ~{MCAS2}: now also R20.1; no longer R19.1
- net ~{MCAS3}: now also R21.1; no longer R18.1
- net ~{MRAS01}: now also R16.1; no longer R17.1
- net ~{MRAS23}: now also R17.1; no longer R16.1
- net ~{RCAS0}: now also J1.2 (~{CAS}), J1.28 (~{CASP}), R18.2; no longer J4.2 (~{CAS}), J4.28 (~{CASP}), R21.2
- net ~{RCAS1}: now also J2.2 (~{CAS}), J2.28 (~{CASP}), R19.2; no longer J3.2 (~{CAS}), J3.28 (~{CASP}), R20.2
- net ~{RCAS2}: now also J3.2 (~{CAS}), J3.28 (~{CASP}), R20.2; no longer J2.2 (~{CAS}), J2.28 (~{CASP}), R19.2
- net ~{RCAS3}: now also J4.2 (~{CAS}), J4.28 (~{CASP}), R21.2; no longer J1.2 (~{CAS}), J1.28 (~{CASP}), R18.2
- net ~{RRAS01}: now also J1.27 (~{RAS}), J2.27 (~{RAS}), R16.2; no longer J3.27 (~{RAS}), J4.27 (~{RAS}), R17.2
- net ~{RRAS23}: now also J3.27 (~{RAS}), J4.27 (~{RAS}), R17.2; no longer J1.27 (~{RAS}), J2.27 (~{RAS}), R16.2
- net MDP02 renamed DP_HI
- net MDP13 renamed DP_LO
- net ~{SMEMR} renamed ~{MEMR}
Other:
- moved on the sheet: J1, J2, J3, J4, R1, R10, R11, R12, R16, R17, R18, R19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
