File: KiCad/isa_slots_power.kicad_sch (KiCad schematic)
At the start: 82 parts, among them J1 BUSAT_HOST, J12 Power, J2 BUSAT_HOST, J3 BUSAT_HOST, J4 BUSAT_HOST, J5 BUSAT_HOST, J6 BUSAT_HOST, U10 LM7905, U8 74HCT14, U9 74HCT74

Commit message: Fix the ROM /OE issue; Update DRAM banks
Connect Flash ROM /OE to ISA /MEMR
Update DRAM banks numbers (swap Bank 0 and Bank 1)
Update chipset DRAM signal names
Renumber DRAM termination resistors according to the signal names
Renumber SIMM and ISA slots, so that they are numbered top to bottom
Parts:
- renumbered J1 to J10, J4 to J7, J3 to J8, J2 to J9
Other:
- moved on the sheet: J10, J5, J6, J7, J8, J9

Commit message: Renumber electrolytic capacitors; use 22 kohm resistor for R39; relocate C9.
Renumber electrolytic capacitors, so that the reference numbers increase from the top of the PCB to the bottom
Use 22 kohm resistor for R39
Relocate C9
Parts:
- C21: value 100uF -> 100nF
- R39: value 20k -> 22k
- renumbered C40 to C27, C38 to C28, C39 to C29, C36 to C30, C37 to C31, C34 to C32, C35 to C33, C33 to C34, C30 to C35, C31 to C36, C32 to C37, C27 to C38, C28 to C39, C29 to C40, C43 to C42, C42 to C43, C46 to C45, C45 to C46, C49 to C48, C48 to C49, RN3 to RN2, RN2 to RN3
Other:
- moved on the sheet: C27, C28, C29, C30, C31, C32, C33, C34, C35, C36, C37, C38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
